File: esp_2fa_board_design.sch (KiCad schematic (older format))
At the start: 50 parts, among them IC1 TPS22919DCKR, J1 Conn_01x06_Female, J2 TYPE-C-31-M-17, J3 Conn_01x02_Male, Q1 DMP2305U-7, SW1 SW_Push, SW2 SW_Push, SW3 BOOT, SW4 RESET, U1 ESP32-WROOM-32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

Commit message: Partially completed rerouting
Parts:
- removed J3: Conn_01x02_Male, Connector_PinHeader_1.27mm:PinHeader_1x01_P1.27mm_Horizontal, symbol Connector:Conn_01x02_Male
- added J3: Conn_01x02_Female, Connector_PinHeader_1.27mm:PinHeader_1x02_P1.27mm_Vertical, symbol Connector:Conn_01x02_Female
- added SW5: POWER SWITCH, Button_Switch_THT:SW_Slide_1P2T_CK_OS102011MS2Q, symbol Switch:SW_DIP_x01
Connections:
- wire segments 188 -> 189
Changed lines of the file:
@@
 Connection ~ 13250 6200
-Wire Wire Line
-	12000 5800 12550 5800
 Wire Wire Line
 	13000 6350 13000 6200
@@
 Wire Wire Line
 	12550 6350 12550 5800
-Connection ~ 12550 5800
 Wire Wire Line
 	12550 5800 13000 5800
@@
 Wire Notes Line width 20 style dash_dot rgb(194, 24, 3)
 	11150 7700 11150 11150
-Text Label 12000 5800 0    50   ~ 0
+Text Label 11450 5800 0    50   ~ 0
 V_INPUT
 Wire Wire Line
@@
 	8650 8700 8650 9300
 Wire Wire Line
-	12750 1550 12750 2150
-Wire Wire Line
 	9450 8700 9450 9300
 Wire Wire Line
@@
 Text Label 10100 9300 1    39   ~ 0
 V_INPUT
-$Comp
-L Connector:Conn_01x02_Male J3
-U 1 1 5FBB5A90
-P 12750 1350
-F 0 "J3" V 12812 1394 50  0000 L CNN
-F 1 "Conn_01x02_Male" V 12903 1394 50  0000 L CNN
-F 2 "Connector_PinHeader_1.27mm:PinHeader_1x01_P1.27mm_Horizontal" H 12750 1350 50  0001 C CNN
-F 3 "~" H 12750 1350 50  0001 C CNN
-	1    12750 1350
-	0    1    1    0
-$EndComp
-Wire Wire Line
-	12650 1550 12650 2150
 Wire Wire Line
 	12450 2150 12650 2150
@@
 	1    0    0    -1
 $EndComp
+$Comp
+L Switch:SW_DIP_x01 SW5
+U 1 1 5FBA599A
+P 12150 5800
+F 0 "SW5" H 12150 6067 50  0000 C CNN
+F 1 "POWER SWITCH" H 12150 5976 50  0000 C CNN
+F 2 "Button_Switch_THT:SW_Slide_1P2T_CK_OS102011MS2Q" H 12150 5800 50  0001 C CNN
+F 3 "~" H 12150 5800 50  0001 C CNN
+	1    12150 5800
+	1    0    0    -1
+$EndComp
+Wire Wire Line
+	12450 5800 12550 5800
+Connection ~ 12550 5800
+Wire Wire Line
+	11850 5800 11450 5800
+$Comp
+L Connector:Conn_01x02_Female J3
+U 1 1 5FBD9746
+P 12650 1100
+F 0 "J3" V 12588 912 50  0000 R CNN
+F 1 "Conn_01x02_Female" V 12497 912 50  0000 R CNN
+F 2 "Connector_PinHeader_1.27mm:PinHeader_1x02_P1.27mm_Vertical" H 12650 1100 50  0001 C CNN
+F 3 "~" H 12650 1100 50  0001 C CNN
+	1    12650 1100
+	0    -1   -1   0
+$EndComp
+Wire Wire Line
+	12650 1300 12650 2150
+Wire Wire Line
+	12750 1300 12750 2150
 $EndSCHEMATC

Commit message: Partially completed routing, regulator section remains
Parts:
- removed J1: Conn_01x06_Female, Connector_PinHeader_2.00mm:PinHeader_1x06_P2.00mm_Vertical, symbol esp_2fa_board_design-rescue:Conn_01x06_Female-Connector
- added J1: Conn_01x02_Female, Connector_PinHeader_1.27mm:PinHeader_1x02_P1.27mm_Vertical, symbol Connector:Conn_01x02_Female
Connections:
- net RX: now also J1.2 (Pin_2)
- net TX: now also J1.1 (Pin_1)
- no-connect marks 28 -> 25
Changed lines of the file:
@@
-	0    -1   -1   0
-$EndComp
-$Comp
-L esp_2fa_board_design-rescue:Conn_01x06_Female-Connector J1
-U 1 1 5F48EBEC
-P 5000 1250
-F 0 "J1" H 4892 725 50  0000 C CNN
-F 1 "Conn_01x06_Female" H 4892 816 50  0000 C CNN
-F 2 "Connector_PinHeader_2.00mm:PinHeader_1x06_P2.00mm_Vertical" H 5000 1250 50  0001 C CNN
-F 3 "~" H 5000 1250 50  0001 C CNN
-	1    5000 1250
 	0    -1   -1   0
 $EndComp
@@
 Text Notes 4550 2400 0    118  ~ 0
 Load Switch
-$Comp
-L esp_2fa_board_design-rescue:GND-power #PWR09
-U 1 1 5FA65CB2
-P 5300 1650
-F 0 "#PWR09" H 5300 1400 50  0001 C CNN
-F 1 "GND" H 5305 1477 50  0000 C CNN
-F 2 "" H 5300 1650 50  0001 C CNN
-F 3 "" H 5300 1650 50  0001 C CNN
-	1    5300 1650
-	1    0    0    -1
-$EndComp
-Wire Wire Line
-	5300 1450 5300 1650
 Wire Wire Line
 	2150 1500 2500 1500
@@
 RX
 Wire Wire Line
-	4900 1450 4900 1700
-Wire Wire Line
-	5000 1450 5000 1700
-Text Label 4900 1700 1    39   ~ 0
+	4950 1250 4950 1500
+Wire Wire Line
+	5050 1250 5050 1500
+Text Label 4950 1500 1    39   ~ 0
 TX
-Text Label 5000 1700 1    39   ~ 0
+Text Label 5050 1500 1    39   ~ 0
 RX
 Wire Wire Line
@@
 NoConn ~ 2150 3500
 NoConn ~ 2150 3600
-NoConn ~ 4800 1450
-NoConn ~ 5100 1450
-NoConn ~ 5200 1450
 NoConn ~ 8300 2500
 NoConn ~ 9300 2400
@@
 Wire Wire Line
 	9950 2150 9950 2050
+Wire Wire Line
+	3150 1000 3100 1000
+Wire Wire Line
+	3450 1000 3500 1000
+$Comp
+L power:GND #PWR033
+U 1 1 5FC88584
+P 3600 1150
+F 0 "#PWR033" H 3600 900 50  0001 C CNN
+F 1 "GND" V 3605 1022 50  0000 R CNN
+F 2 "" H 3600 1150 50  0001 C CNN
+F 3 "" H 3600 1150 50  0001 C CNN
+	1    3600 1150
+	0    -1   -1   0
+$EndComp
+Wire Wire Line
+	3100 1000 3100 1150
+Wire Wire Line
+	3100 1300 3150 1300
+Wire Wire Line
+	3450 1300 3500 1300
+Connection ~ 3500 1150
+Wire Wire Line
+	3500 1150 3500 1300
+Wire Wire Line
+	3500 1000 3500 1150
+Wire Wire Line
+	1550 1150 3100 1150
+Connection ~ 3100 1150
+Wire Wire Line
+	3100 1150 3100 1300
+Text Notes 14850 2700 0    50   ~ 0
+ON - Charge complete state\nOFF- Charging state
+Text Notes 11550 4100 0    79   ~ 0
+I_charge = 1000/R_PROG\nI_charge = 1000/4700 = 213 mA\n\nWhere:\nR_PROG = kOhms\nI_REG = milliampere
+Wire Wire Line
+	3950 8900 3950 9200
+Connection ~ 3950 9200
+Wire Wire Line
+	3200 9200 3600 9200
+Connection ~ 1550 1150
+Wire Wire Line
+	1550 1150 1550 1200
+Wire Wire Line
+	1550 1050 1550 1150
+Wire Wire Line
+	3600 1150 3500 1150
+$Comp
+L Connector:TestPoint TP7
+U 1 1 5FBABC3C
+P 8200 8700
+F 0 "TP7" H 8258 8818 50  0000 L CNN
+F 1 "OLED_SCL" H 8258 8727 50  0000 L CNN
+F 2 "Connector_Wire:SolderWirePad_1x01_SMD_1x2mm" H 8400 8700 50  0001 C CNN
+F 3 "~" H 8400 8700 50  0001 C CNN
+	1    8200 8700
+	1    0    0    -1
+$EndComp
+$Comp
+L Connector:TestPoint TP6
+U 1 1 5FBABFAB
+P 7750 8700
+F 0 "TP6" H 7808 8818 50  0000 L CNN
+F 1 "OLED_SDA" H 7808 8727 50  0000 L CNN
+F 2 "Connector_Wire:SolderWirePad_1x01_SMD_1x2mm" H 7950 8700 50  0001 C CNN
+F 3 "~" H 7950 8700 50  0001 C CNN
+	1    7750 8700
+	1    0    0    -1
+$EndComp
+$Comp
+L Connector:TestPoint TP3
+U 1 1 5FBAC272
+P 7300 8700
+F 0 "TP3" H 7358 8818 50  0000 L CNN
+F 1 "RTC_SCL" H 7358 8727 50  0000 L CNN
+F 2 "Connector_Wire:SolderWirePad_1x01_SMD_1x2mm" H 7500 8700 50  0001 C CNN
+F 3 "~" H 7500 8700 50  0001 C CNN
+	1    7300 8700
+	1    0    0    -1
+$EndComp
+$Comp
+L Connector:TestPoint TP2
+U 1 1 5FBAC716
+P 6900 8700
+F 0 "TP2" H 6958 8818 50  0000 L CNN
+F 1 "RTC_SDA" H 6958 8727 50  0000 L CNN
+F 2 "Connector_Wire:SolderWirePad_1x01_SMD_1x2mm" H 7100 8700 50  0001 C CNN
+F 3 "~" H 7100 8700 50  0001 C CNN
+	1    6900 8700
+	1    0    0    -1
+$EndComp
+Wire Wire Line
+	8200 8700 8200 9300
+Wire Wire Line
+	7750 8700 7750 9300
+Wire Wire Line
+	7300 8700 7300 9300
+Wire Wire Line
+	6900 8700 6900 9300
+Text Label 6900 9300 1    50   ~ 0
+IO5_SDA
+Text Label 7300 9300 1    50   ~ 0
+IO18_SCL
+Text Label 7750 9300 1    50   ~ 0
+IO21_SDA
+Text Label 8200 9300 1    50   ~ 0
+IO22_SCL
+$Comp
+L Connector:TestPoint TP8
+U 1 1 5FC0B51C
+P 9050 8700
+F 0 "TP8" H 9108 8818 50  0000 L CNN
+F 1 "GND" H 9108 8727 50  0000 L CNN
+F 2 "Connector_Wire:SolderWirePad_1x01_SMD_1x2mm" H 9250 8700 50  0001 C CNN
+F 3 "~" H 9250 8700 50  0001 C CNN
+	1    9050 8700
+	1    0    0    -1
+$EndComp
+Wire Wire Line
+	9050 8700 9050 9300
+$Comp
+L power:GND #PWR034
+U 1 1 5FC15BFB
+P 9050 9300
+F 0 "#PWR034" H 9050 9050 50  0001 C CNN
+F 1 "GND" H 9055 9127 50  0000 C CNN
+F 2 "" H 9050 9300 50  0001 C CNN
+F 3 "" H 9050 9300 50  0001 C CNN
+	1    9050 9300
+	1    0    0    -1
+$EndComp
+$Comp
+L Switch:SW_DIP_x01 SW5
+U 1 1 5FBA599A
+P 12150 5800
+F 0 "SW5" H 12150 6067 50  0000 C CNN
+F 1 "POWER SWITCH" H 12150 5976 50  0000 C CNN
+F 2 "Button_Switch_THT:SW_Slide_1P2T_CK_OS102011MS2Q" H 12150 5800 50  0001 C CNN
+F 3 "~" H 12150 5800 50  0001 C CNN
+	1    12150 5800
+	1    0    0    -1
+$EndComp
+Wire Wire Line
+	12450 5800 12550 5800
+Connection ~ 12550 5800
+Wire Wire Line
+	11850 5800 11450 5800
+$Comp
+L Connector:Conn_01x02_Female J3
+U 1 1 5FBD9746
+P 12650 1100
+F 0 "J3" V 12588 912 50  0000 R CNN
+F 1 "Conn_01x02_Female" V 12497 912 50  0000 R CNN
+F 2 "Connector_PinHeader_1.27mm:PinHeader_1x02_P1.27mm_Vertical" H 12650 1100 50  0001 C CNN
+F 3 "~" H 12650 1100 50  0001 C CNN
+	1    12650 1100
+	0    -1   -1   0
+$EndComp
+Wire Wire Line
+	12650 1300 12650 2150
+Wire Wire Line
+	12750 1300 12750 2150
 $Comp
 L esp_2fa_board_design-rescue:C-Device C2
@@
 	0    -1   -1   0
 $EndComp
-Wire Wire Line
-	3150 1000 3100 1000
-Wire Wire Line
-	3450 1000 3500 1000
-$Comp
-L power:GND #PWR033
-U 1 1 5FC88584
-P 3600 1150
-F 0 "#PWR033" H 3600 900 50  0001 C CNN
-F 1 "GND" V 3605 1022 50  0000 R CNN
-F 2 "" H 3600 1150 50  0001 C CNN
-F 3 "" H 3600 1150 50  0001 C CNN
-	1    3600 1150
+$Comp
+L Connector:Conn_01x02_Female J1
+U 1 1 5FC16F81
+P 4950 1050
+F 0 "J1" V 4888 862 50  0000 R CNN
+F 1 "Conn_01x02_Female" V 4797 862 50  0000 R CNN
+F 2 "Connector_PinHeader_1.27mm:PinHeader_1x02_P1.27mm_Vertical" H 4950 1050 50  0001 C CNN
+F 3 "~" H 4950 1050 50  0001 C CNN
+	1    4950 1050
 	0    -1   -1   0
 $EndComp
-Wire Wire Line
-	3100 1000 3100 1150
-Wire Wire Line
-	3100 1300 3150 1300
-Wire Wire Line
-	3450 1300 3500 1300
-Connection ~ 3500 1150
-Wire Wire Line
-	3500 1150 3500 1300
-Wire Wire Line
-	3500 1000 3500 1150
-Wire Wire Line
-	1550 1150 3100 1150
-Connection ~ 3100 1150
-Wire Wire Line
-	3100 1150 3100 1300
-Text Notes 14850 2700 0    50   ~ 0
-ON - Charge complete state\nOFF- Charging state
-Text Notes 11550 4100 0    79   ~ 0
-I_charge = 1000/R_PROG\nI_charge = 1000/4700 = 213 mA\n\nWhere:\nR_PROG = kOhms\nI_REG = milliampere
-Wire Wire Line
-	3950 8900 3950 9200
-Connection ~ 3950 9200
-Wire Wire Line
-	3200 9200 3600 9200
-Connection ~ 1550 1150
-Wire Wire Line
-	1550 1150 1550 1200
-Wire Wire Line
-	1550 1050 1550 1150
-Wire Wire Line
-	3600 1150 3500 1150
-$Comp
-L Connector:TestPoint TP7
-U 1 1 5FBABC3C
-P 8200 8700
-F 0 "TP7" H 8258 8818 50  0000 L CNN
-F 1 "OLED_SCL" H 8258 8727 50  0000 L CNN
-F 2 "Connector_Wire:SolderWirePad_1x01_SMD_1x2mm" H 8400 8700 50  0001 C CNN
-F 3 "~" H 8400 8700 50  0001 C CNN
-	1    8200 8700
-	1    0    0    -1
-$EndComp
-$Comp
-L Connector:TestPoint TP6
-U 1 1 5FBABFAB
-P 7750 8700
-F 0 "TP6" H 7808 8818 50  0000 L CNN
-F 1 "OLED_SDA" H 7808 8727 50  0000 L CNN
-F 2 "Connector_Wire:SolderWirePad_1x01_SMD_1x2mm" H 7950 8700 50  0001 C CNN
-F 3 "~" H 7950 8700 50  0001 C CNN
-	1    7750 8700
-	1    0    0    -1
-$EndComp
-$Comp
-L Connector:TestPoint TP3
-U 1 1 5FBAC272
-P 7300 8700
-F 0 "TP3" H 7358 8818 50  0000 L CNN
-F 1 "RTC_SCL" H 7358 8727 50  0000 L CNN
-F 2 "Connector_Wire:SolderWirePad_1x01_SMD_1x2mm" H 7500 8700 50  0001 C CNN
-F 3 "~" H 7500 8700 50  0001 C CNN
-	1    7300 8700
-	1    0    0    -1
-$EndComp
-$Comp
-L Connector:TestPoint TP2
-U 1 1 5FBAC716
-P 6900 8700
-F 0 "TP2" H 6958 8818 50  0000 L CNN
-F 1 "RTC_SDA" H 6958 8727 50  0000 L CNN
-F 2 "Connector_Wire:SolderWirePad_1x01_SMD_1x2mm" H 7100 8700 50  0001 C CNN
-F 3 "~" H 7100 8700 50  0001 C CNN
-	1    6900 8700
-	1    0    0    -1
-$EndComp
-Wire Wire Line
-	8200 8700 8200 9300
-Wire Wire Line
-	7750 8700 7750 9300
-Wire Wire Line
-	7300 8700 7300 9300
-Wire Wire Line
-	6900 8700 6900 9300
-Text Label 6900 9300 1    50   ~ 0
-IO5_SDA
-Text Label 7300 9300 1    50   ~ 0
-IO18_SCL
-Text Label 7750 9300 1    50   ~ 0
-IO21_SDA
-Text Label 8200 9300 1    50   ~ 0
-IO22_SCL
-$Comp
-L Connector:TestPoint TP8
-U 1 1 5FC0B51C
-P 9050 8700
-F 0 "TP8" H 9108 8818 50  0000 L CNN
-F 1 "GND" H 9108 8727 50  0000 L CNN
-F 2 "Connector_Wire:SolderWirePad_1x01_SMD_1x2mm" H 9250 8700 50  0001 C CNN
-F 3 "~" H 9250 8700 50  0001 C CNN
-	1    9050 8700
-	1    0    0    -1
-$EndComp
-Wire Wire Line
-	9050 8700 9050 9300
-$Comp
-L power:GND #PWR034
-U 1 1 5FC15BFB
-P 9050 9300
-F 0 "#PWR034" H 9050 9050 50  0001 C CNN
-F 1 "GND" H 9055 9127 50  0000 C CNN
-F 2 "" H 9050 9300 50  0001 C CNN
-F 3 "" H 9050 9300 50  0001 C CNN
-	1    9050 9300
-	1    0    0    -1
-$EndComp
-$Comp
-L Switch:SW_DIP_x01 SW5
-U 1 1 5FBA599A
-P 12150 5800
-F 0 "SW5" H 12150 6067 50  0000 C CNN
-F 1 "POWER SWITCH" H 12150 5976 50  0000 C CNN
-F 2 "Button_Switch_THT:SW_Slide_1P2T_CK_OS102011MS2Q" H 12150 5800 50  0001 C CNN
-F 3 "~" H 12150 5800 50  0001 C CNN
-	1    12150 5800
-	1    0    0    -1
-$EndComp
-Wire Wire Line
-	12450 5800 12550 5800
-Connection ~ 12550 5800
-Wire Wire Line
-	11850 5800 11450 5800
-$Comp
-L Connector:Conn_01x02_Female J3
-U 1 1 5FBD9746
-P 12650 1100
-F 0 "J3" V 12588 912 50  0000 R CNN
-F 1 "Conn_01x02_Female" V 12497 912 50  0000 R CNN
-F 2 "Connector_PinHeader_1.27mm:PinHeader_1x02_P1.27mm_Vertical" H 12650 1100 50  0001 C CNN
-F 3 "~" H 12650 1100 50  0001 C CNN
-	1    12650 1100
-	0    -1   -1   0
-$EndComp
-Wire Wire Line
-	12650 1300 12650 2150
-Wire Wire Line
-	12750 1300 12750 2150
 $EndSCHEMATC

Commit message: Updated schematics by adding one more filter capacitor to voltage regulator VIN and changed routing accordingly
Parts:
- added C11: 10uF 50V, Capacitor_SMD:C_1206_3216Metric, symbol esp_2fa_board_design-rescue:C-Device
Connections:
- net GND: now also C11.2
- net at C6.1, R1.1, SW5.2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: now also C11.1
Changed lines of the file:
@@
 Connection ~ 13000 6200
 Wire Wire Line
-	12550 6350 12550 5800
+	12550 6350 12550 6250
 Wire Wire Line
 	12550 5800 13000 5800
@@
 	0    -1   -1   0
 $EndComp
+$Comp
+L esp_2fa_board_design-rescue:C-Device C11
+U 1 1 5FC158D3
+P 12150 6500
+F 0 "C11" H 12265 6546 50  0000 L CNN
+F 1 "10uF 50V" H 12150 6400 50  0000 L CNN
+F 2 "Capacitor_SMD:C_1206_3216Metric" H 12188 6350 50  0001 C CNN
+F 3 "~" H 12150 6500 50  0001 C CNN
+	1    12150 6500
+	1    0    0    -1
+$EndComp
+Wire Wire Line
+	12150 6350 12150 6250
+Wire Wire Line
+	12150 6250 12550 6250
+Connection ~ 12550 6250
+Wire Wire Line
+	12550 6250 12550 5800
+Wire Wire Line
+	12150 6650 12150 6900
+Wire Wire Line
+	12150 6900 12550 6900
+Connection ~ 12550 6900
 $EndSCHEMATC

Commit message: Completed routing pcb
Parts:
- SW1: value SW_Push -> UP
- SW2: value SW_Push -> DOWN
- SW3: value BOOT -> BOOT/SELECT
Changed lines of the file:
@@
 P 1500 6350
 F 0 "SW3" V 1546 6302 50  0000 R CNN
-F 1 "BOOT" V 1455 6302 50  0000 R CNN
+F 1 "BOOT/SELECT" V 1455 6302 50  0000 R CNN
 F 2 "Button_Switch_SMD:SW_Push_1P1T_NO_6x6mm_H9.5mm" H 1500 6550 50  0001 C CNN
 F 3 "~" H 1500 6550 50  0001 C CNN
@@
 P 4900 6350
 F 0 "SW2" V 4946 6302 50  0000 R CNN
-F 1 "SW_Push" V 4855 6302 50  0000 R CNN
+F 1 "DOWN" V 4855 6302 50  0000 R CNN
 F 2 "Button_Switch_SMD:SW_Push_1P1T_NO_6x6mm_H9.5mm" H 4900 6550 50  0001 C CNN
 F 3 "~" H 4900 6550 50  0001 C CNN
@@
 P 4050 6350
 F 0 "SW1" V 4096 6302 50  0000 R CNN
-F 1 "SW_Push" V 4005 6302 50  0000 R CNN
+F 1 "UP" V 4005 6302 50  0000 R CNN
 F 2 "Button_Switch_SMD:SW_Push_1P1T_NO_6x6mm_H9.5mm" H 4050 6550 50  0001 C CNN
 F 3 "~" H 4050 6550 50  0001 C CNN

Commit message: Updated pcb to increase rx/tx header size
Parts:
- J1: footprint Connector_PinHeader_1.27mm:PinHeader_1x02_P1.27mm_Vertical -> Connector_PinHeader_2.54mm:PinHeader_1x02_P2.54mm_Vertical
Changed lines of the file:
@@
 F 0 "J1" V 4888 862 50  0000 R CNN
 F 1 "Conn_01x02_Female" V 4797 862 50  0000 R CNN
-F 2 "Connector_PinHeader_1.27mm:PinHeader_1x02_P1.27mm_Vertical" H 4950 1050 50  0001 C CNN
+F 2 "Connector_PinHeader_2.54mm:PinHeader_1x02_P2.54mm_Vertical" H 4950 1050 50  0001 C CNN
 F 3 "~" H 4950 1050 50  0001 C CNN
 	1    4950 1050

Commit message: Replaced footprint of switch with custom made
Parts:
- SW5: footprint Button_Switch_THT:SW_Slide_1P2T_CK_OS102011MS2Q -> slide_switch_12D00:Slide_Switch_SS-12D00
Changed lines of the file:
@@
 F 0 "SW5" H 12150 6067 50  0000 C CNN
 F 1 "POWER SWITCH" H 12150 5976 50  0000 C CNN
-F 2 "Button_Switch_THT:SW_Slide_1P2T_CK_OS102011MS2Q" H 12150 5800 50  0001 C CNN
+F 2 "slide_switch_12D00:Slide_Switch_SS-12D00" H 12150 5800 50  0001 C CNN
 F 3 "~" H 12150 5800 50  0001 C CNN
 	1    12150 5800
