File: kicad_project/esp_2fa_board_design.sch (KiCad schematic (older format))
At the start: 52 parts, among them IC1 TPS22919DCKR, J1 Conn_01x02_Female, J2 TYPE-C-31-M-17, J3 Conn_01x02_Female, Q1 DMP2305U-7, SW1 UP, SW2 DOWN, SW3 BOOT/SELECT, SW4 RESET, SW5 POWER SWITCH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

Commit message: Updated KiCad project with new path to component libraries
Parts:
- BT1: symbol esp_2fa_board_design-rescue:Battery_Cell-Device -> esp_2fa_board_design-rescue:Battery_Cell-Device-esp_2fa_board_design-rescue
- C1, C10, C11, C2, C3, C4, C5, C6, C7, C8, C9: symbol esp_2fa_board_design-rescue:C-Device -> esp_2fa_board_design-rescue:C-Device-esp_2fa_board_design-rescue
- D2: symbol esp_2fa_board_design-rescue:LED-Device -> esp_2fa_board_design-rescue:LED-Device-esp_2fa_board_design-rescue
- D3: symbol esp_2fa_board_design-rescue:1N5819-Diode -> esp_2fa_board_design-rescue:1N5819-Diode-esp_2fa_board_design-rescue
- L1: symbol esp_2fa_board_design-rescue:INDUCTOR-pspice -> esp_2fa_board_design-rescue:INDUCTOR-pspice-esp_2fa_board_design-rescue
- R1, R10, R11, R12, R13, R14, R2, R3, R4, R5, R6, R7, R8, R9: symbol esp_2fa_board_design-rescue:R_Small_US-Device -> esp_2fa_board_design-rescue:R_Small_US-Device-esp_2fa_board_design-rescue
- SW1, SW2, SW3, SW4: symbol esp_2fa_board_design-rescue:SW_Push-Switch -> esp_2fa_board_design-rescue:SW_Push-Switch-esp_2fa_board_design-rescue
- U1: symbol esp_2fa_board_design-rescue:ESP32-WROOM-32-RF_Module -> esp_2fa_board_design-rescue:ESP32-WROOM-32-RF_Module-esp_2fa_board_design-rescue
- U2: symbol esp_2fa_board_design-rescue:DS3231M-Timer_RTC -> esp_2fa_board_design-rescue:DS3231M-Timer_RTC-esp_2fa_board_design-rescue
- U3: symbol esp_2fa_board_design-rescue:MCP73831-2-OT-Battery_Management -> esp_2fa_board_design-rescue:MCP73831-2-OT-Battery_Management-esp_2fa_board_design-rescue
- U4: symbol esp_2fa_board_design-rescue:TPS63001-Regulator_Switching -> esp_2fa_board_design-rescue:TPS63001-Regulator_Switching-esp_2fa_board_design-rescue
